Commit message: Tuned parameters and weights for walking taks

File: robots/go2_robot_sdk/urdf/go2_no_limit.urdf (robot description, URDF)
Before this commit: robot go2, 33 links, 32 joints
Joints:
- joint FL_calf_joint: limit lower=-10 upper=10 effort=1000 velocity=1000 -> (none)
- joint FL_hip_joint: limit lower=-10 upper=10 effort=1000 velocity=1000 -> (none)
- joint FL_thigh_joint: limit lower=-10 upper=10 effort=1000 velocity=1000 -> (none)
- joint FR_calf_joint: limit lower=-10 upper=10 effort=1000 velocity=1000 -> (none)
- joint FR_hip_joint: limit lower=-10 upper=10 effort=1000 velocity=1000 -> (none)
- joint FR_thigh_joint: limit lower=-10 upper=10 effort=1000 velocity=1000 -> (none)
- joint RL_calf_joint: limit lower=-10 upper=10 effort=1000 velocity=1000 -> (none)
- joint RL_hip_joint: limit lower=-10 upper=10 effort=1000 velocity=1000 -> (none)
- joint RL_thigh_joint: limit lower=-10 upper=10 effort=1000 velocity=1000 -> (none)
- joint RR_calf_joint: limit lower=-10 upper=10 effort=1000 velocity=1000 -> (none)
- joint RR_hip_joint: limit lower=-10 upper=10 effort=1000 velocity=1000 -> (none)
- joint RR_thigh_joint: limit lower=-10 upper=10 effort=1000 velocity=1000 -> (none)
