Commit message: update CMAKE to include all mujoco version. bump c++ standard. model verification in progress

File: robots/trifinger/trifinger.urdf (robot description, URDF)
Before this commit: robot trifinger, 17 links, 16 joints
Links:
- link finger0_base_link: geometry collision mesh filename=package://trifinger/meshes/base_back.stl; collision mesh filename=package://trifinger/meshes/base_front.stl
- link finger0_lower_link: geometry collision mesh filename=package://trifinger/meshes/lower_link.stl; visual mesh filename=package://trifinger/meshes/lower_link.stl
- link finger0_middle_link: geometry collision mesh filename=package://trifinger/meshes/middle_link.stl; visual mesh filename=package://trifinger/meshes/middle_link.stl
- link finger0_upper_link: geometry collision mesh filename=package://trifinger/meshes/upper_link.stl; visual mesh filename=package://trifinger/meshes/upper_link.stl
- link finger1_base_link: geometry collision mesh filename=package://trifinger/meshes/base_back.stl; collision mesh filename=package://trifinger/meshes/base_front.stl
- link finger1_lower_link: geometry collision mesh filename=package://trifinger/meshes/lower_link.stl; visual mesh filename=package://trifinger/meshes/lower_link.stl
- link finger1_middle_link: geometry collision mesh filename=package://trifinger/meshes/middle_link.stl; visual mesh filename=package://trifinger/meshes/middle_link.stl
- link finger1_upper_link: geometry collision mesh filename=package://trifinger/meshes/upper_link.stl; visual mesh filename=package://trifinger/meshes/upper_link.stl
- link finger2_base_link: geometry collision mesh filename=package://trifinger/meshes/base_back.stl; collision mesh filename=package://trifinger/meshes/base_front.stl
- link finger2_lower_link: geometry collision mesh filename=package://trifinger/meshes/lower_link.stl; visual mesh filename=package://trifinger/meshes/lower_link.stl
- link finger2_middle_link: geometry collision mesh filename=package://trifinger/meshes/middle_link.stl; visual mesh filename=package://trifinger/meshes/middle_link.stl
- link finger2_upper_link: geometry collision mesh filename=package://trifinger/meshes/upper_link.stl; visual mesh filename=package://trifinger/meshes/upper_link.stl
