Commit message: Updated URDF, Added new URDF and XML, updated robot envrionment

File: robots/trifinger/trifinger_scene.urdf (robot description, URDF)
Before this commit: robot trifinger, 17 links, 16 joints
Links:
- added link ground_link, mass 1; collision box size=20 20 0.1; visual box size=20 20 0.1
Joints:
- added joint base_to_ground_joint: type fixed, parent base_link, child ground_link, origin xyz=0 0 0 rpy=0 0 0

Commit message: refactored trifinger env - now everything works properly

File: robots/trifinger/trifinger_scene.urdf (robot description, URDF)
Before this commit: robot trifinger_with_ground, 18 links, 17 joints
Links:
- removed link finger0_base_link
- removed link finger0_lower_link
- removed link finger0_middle_link
- removed link finger0_tip_link
- removed link finger0_upper_link
- removed link finger1_base_link
- removed link finger1_lower_link
- removed link finger1_middle_link
- removed link finger1_tip_link
- removed link finger1_upper_link
- removed link finger2_base_link
- removed link finger2_lower_link
- removed link finger2_middle_link
- removed link finger2_tip_link
- removed link finger2_upper_link
- removed link ground_link
- removed link trifinger_base_link
- added link boundary_link, mass 2; collision mesh filename=package://meshes/high_table_boundary.stl scale=1 1 1; visual mesh filename=package://meshes/high_table_boundary.stl scale=1 1 1
- added link finger_base_link_0, mass 1; collision mesh filename=package://meshes/SIM__BL-Finger_Base.stl scale=1 1 1; visual mesh filename=package://meshes/SIM__BL-Finger_Base.stl scale=1 1 1
- added link finger_base_link_120, mass 1; collision mesh filename=package://meshes/SIM__BL-Finger_Base.stl scale=1 1 1; visual mesh filename=package://meshes/SIM__BL-Finger_Base.stl scale=1 1 1
- added link finger_base_link_240, mass 1; collision mesh filename=package://meshes/SIM__BL-Finger_Base.stl scale=1 1 1; visual mesh filename=package://meshes/SIM__BL-Finger_Base.stl scale=1 1 1
- added link finger_lower_link_0, mass 0.01; collision mesh filename=package://meshes/SIM_BL_FINGER_TIP_LINK.stl scale=1 1 1; visual mesh filename=package://meshes/SIM_BL_FINGER_TIP_LINK.stl scale=1 1 1
- added link finger_lower_link_120, mass 0.01; collision mesh filename=package://meshes/SIM_BL_FINGER_TIP_LINK.stl scale=1 1 1; visual mesh filename=package://meshes/SIM_BL_FINGER_TIP_LINK.stl scale=1 1 1
- added link finger_lower_link_240, mass 0.01; collision mesh filename=package://meshes/SIM_BL_FINGER_TIP_LINK.stl scale=1 1 1; visual mesh filename=package://meshes/SIM_BL_FINGER_TIP_LINK.stl scale=1 1 1
- added link finger_middle_link_0, mass 0.2; collision mesh filename=package://meshes/SIM__BL-Finger_Intermediate.stl scale=1 1 1; visual mesh filename=package://meshes/SIM__BL-Finger_Intermediate.stl scale=1 1 1
- added link finger_middle_link_120, mass 0.2; collision mesh filename=package://meshes/SIM__BL-Finger_Intermediate.stl scale=1 1 1; visual mesh filename=package://meshes/SIM__BL-Finger_Intermediate.stl scale=1 1 1
- added link finger_middle_link_240, mass 0.2; collision mesh filename=package://meshes/SIM__BL-Finger_Intermediate.stl scale=1 1 1; visual mesh filename=package://meshes/SIM__BL-Finger_Intermediate.stl scale=1 1 1
- added link finger_tip_link_0, mass 0.02
- added link finger_tip_link_120, mass 0.02
- added link finger_tip_link_240, mass 0.02
- added link finger_upper_link_0, mass 0.2; collision mesh filename=package://meshes/SIM__BL-Finger_Proximal.stl scale=1 1 1; visual mesh filename=package://meshes/SIM__BL-Finger_Proximal.stl scale=1 1 1
- added link finger_upper_link_120, mass 0.2; collision mesh filename=package://meshes/SIM__BL-Finger_Proximal.stl scale=1 1 1; visual mesh filename=package://meshes/SIM__BL-Finger_Proximal.stl scale=1 1 1
- added link finger_upper_link_240, mass 0.2; collision mesh filename=package://meshes/SIM__BL-Finger_Proximal.stl scale=1 1 1; visual mesh filename=package://meshes/SIM__BL-Finger_Proximal.stl scale=1 1 1
- added link table_link, mass 2; collision mesh filename=package://meshes/trifinger_table_without_border.stl scale=1 1 1; visual mesh filename=package://meshes/trifinger_table_without_border.stl scale=1 1 1
- added link upper_holder_link, mass 1
Joints:
- removed joint base_to_ground_joint
- removed joint base_to_trifinger_base_joint
- removed joint finger0_base_to_upper_joint
- removed joint finger0_lower_to_tip_joint
- removed joint finger0_middle_to_lower_joint
- removed joint finger0_upper_to_middle_joint
- removed joint finger1_base_to_upper_joint
- removed joint finger1_lower_to_tip_joint
- removed joint finger1_middle_to_lower_joint
- removed joint finger1_upper_to_middle_joint
- removed joint finger2_base_to_upper_joint
- removed joint finger2_lower_to_tip_joint
- removed joint finger2_middle_to_lower_joint
- removed joint finger2_upper_to_middle_joint
- removed joint trifinger_base_to_finger0_joint
- removed joint trifinger_base_to_finger1_joint
- removed joint trifinger_base_to_finger2_joint
- added joint base_to_table: type fixed, parent base_link, child table_link, origin xyz=0 0 0
- added joint base_to_upper_holder_joint: type fixed, parent base_link, child upper_holder_link, origin xyz=0 0 0.29
- added joint finger_base_to_upper_joint_0: type revolute, parent finger_base_link_0, child finger_upper_link_0, origin xyz=0 0 0 rpy=0 0 0, axis 0 1 0, limit lower=-1.5707963267948966 upper=1.5707963267948966 effort=1000 velocity=1000
- added joint finger_base_to_upper_joint_120: type revolute, parent finger_base_link_120, child finger_upper_link_120, origin xyz=0 0 0 rpy=0 0 0, axis 0 1 0, limit lower=-1.5707963267948966 upper=1.5707963267948966 effort=1000 velocity=1000
- added joint finger_base_to_upper_joint_240: type revolute, parent finger_base_link_240, child finger_upper_link_240, origin xyz=0 0 0 rpy=0 0 0, axis 0 1 0, limit lower=-1.5707963267948966 upper=1.5707963267948966 effort=1000 velocity=1000
- added joint finger_lower_to_tip_joint_0: type fixed, parent finger_lower_link_0, child finger_tip_link_0, origin xyz=0 0 -0.16
- added joint finger_lower_to_tip_joint_120: type fixed, parent finger_lower_link_120, child finger_tip_link_120, origin xyz=0 0 -0.16
- added joint finger_lower_to_tip_joint_240: type fixed, parent finger_lower_link_240, child finger_tip_link_240, origin xyz=0 0 -0.16
- added joint finger_middle_to_lower_joint_0: type revolute, parent finger_middle_link_0, child finger_lower_link_0, origin xyz=0 0 -0.16 rpy=0 0 0, axis 1 0 0, limit lower=-3.001966313430247 upper=3.001966313430247 effort=1000 velocity=1000
- added joint finger_middle_to_lower_joint_120: type revolute, parent finger_middle_link_120, child finger_lower_link_120, origin xyz=0 0 -0.16 rpy=0 0 0, axis 1 0 0, limit lower=-3.001966313430247 upper=3.001966313430247 effort=1000 velocity=1000
- added joint finger_middle_to_lower_joint_240: type revolute, parent finger_middle_link_240, child finger_lower_link_240, origin xyz=0 0 -0.16 rpy=0 0 0, axis 1 0 0, limit lower=-3.001966313430247 upper=3.001966313430247 effort=1000 velocity=1000
- added joint finger_upper_to_middle_joint_0: type revolute, parent finger_upper_link_0, child finger_middle_link_0, origin xyz=0 0 0 rpy=0 0 0, axis -1 0 0, limit lower=-1.3526301702956054 upper=4.494222823885399 effort=1000 velocity=1000
- added joint finger_upper_to_middle_joint_120: type revolute, parent finger_upper_link_120, child finger_middle_link_120, origin xyz=0 0 0 rpy=0 0 0, axis -1 0 0, limit lower=-1.3526301702956054 upper=4.494222823885399 effort=1000 velocity=1000
- added joint finger_upper_to_middle_joint_240: type revolute, parent finger_upper_link_240, child finger_middle_link_240, origin xyz=0 0 0 rpy=0 0 0, axis -1 0 0, limit lower=-1.3526301702956054 upper=4.494222823885399 effort=1000 velocity=1000
- added joint holder_to_finger_0: type fixed, parent upper_holder_link, child finger_base_link_0, origin xyz=0.0 0.04 0 rpy=0 0 0
- added joint holder_to_finger_120: type fixed, parent upper_holder_link, child finger_base_link_120, origin xyz=0.034641016151377546 -0.01999999999999999 0 rpy=0 0 -2.0943951023931953
- added joint holder_to_finger_240: type fixed, parent upper_holder_link, child finger_base_link_240, origin xyz=-0.03464101615137754 -0.020000000000000018 0 rpy=0 0 -4.1887902047863905
- added joint table_to_boundary: type fixed, parent table_link, child boundary_link, origin xyz=0 0 0
