Commit message: Updated urdf and xml

File: robots/trifinger/trifinger_cube_scene.urdf (robot description, URDF)
Before this commit: robot trifinger_scene, 20 links, 19 joints
Links:
- removed link cube
- added link cube_link, mass 0.1; collision box size=0.025 0.025 0.025; visual box size=0.05 0.05 0.05
Joints:
- removed joint root_joint
- added joint cube_joint: type floating, parent world, child cube_link, origin xyz=0 0 0.00 rpy=0 0 0

Commit message: Updated XML and URDF

File: robots/trifinger/trifinger_cube_scene.urdf (robot description, URDF)
Before this commit: robot trifinger_scene, 20 links, 19 joints
Links:
- removed link boundary_link
Joints:
- removed joint table_to_boundary
